Commit message: Project 3 Lab until rviz

File: catkin_ws/src/my_robot/urdf/my_robot.xacro (robot description, xacro)
@@ -22,12 +22,18 @@
       <origin xyz="0 0 0" rpy=" 0 0 0"/>
       <geometry>
-        <box size=".4 .2 .1"/>
+        <cylinder radius="0.1" length="0.05"/>
       </geometry>
+      <material name ="Cyan">
+        <color rgba="0 1.0 1.0 1.0"/>
+      </material>
     </collision>
     <visual name='chassis_visual'>
       <origin xyz="0 0 0" rpy=" 0 0 0"/>
       <geometry>
-        <box size=".4 .2 .1"/>
+        <cylinder radius="0.1" length="0.05"/>
       </geometry>
+      <material name ="Cyan">
+        <color rgba="0 1.0 1.0 1.0"/>
+      </material>
     </visual>
     <collision name='back_caster_collision'>
